File: LC-Meter.kicad_pcb (KiCad board)
At the start: 2 copper layers, 134.5 x 83.9 mm, 27 parts, among them J1 Cx/Lx, J2 Power in, Q1 BC547, SW1 SW_Slide_DPDT, U1 LM311

Commit message: UpDate
Other:
- board text added: "youtube.com/@TeknoTrek"
