File: LC-Meter.kicad_sch (KiCad schematic)
At the start: 27 parts, among them J1 Cx/Lx, J2 Power in, Q1 BC547, SW1 SW_Slide_DPDT, U1 LM311

Commit message: UpDate
Other:
- note added: "LC METER"
- note added: "LC Meter build video: https://www.youtube.com/watch?v=YbbpxDlLRkQ"
- note added: "youtube.com/@TeknoTrek"
- moved on the sheet: A1, C1, C2, C3, C4, D1, J1, J2, JP1, JP2, L1, Q1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
